File: pcb/afe.kicad_sch (KiCad schematic)
At the start: 0 parts

Commit message: Update paper with latest architecture, add openEMS EM simulations (RF, SI, PDN), update schematics with real symbols/wires, add 3D models and openEMS figures
Other:
- note removed: "Eight DAC thresholds; RC filtering at each comparator; optional buffered analog monitor/test points"
- note removed: "OPA858 supply/bias must satisfy common-mode and output swing across tolerance; old 3V3/VBOT circuit rejected"
- note removed: "Repeat x4: touch-safe panel input -> low-capacitance protection -> OPA858 TIA"
- note removed: "Summing-node no-pour keepout and extracted-parasitic stability simulation are release gates"
- note removed: "TIA output -> low-threshold comparator + high-threshold comparator -> active-low FPGA inputs"
Changed lines of the file:
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@@
-(kicad_sch (version 20250114) (generator "eeschema") (generator_version "9.0")
- (paper "A3")
-  (title_block (title "Muon3 four-channel analog front end") (date "2026-07-11") (rev "P0") (comment 1 "ARCHITECTURE - electrical capture pending"))
-  (text "Repeat x4: touch-safe panel input -> low-capacitance protection -> OPA858 TIA" (at 25 35 0) (effects (font (size 2 2)) (justify left)))
-  (text "OPA858 supply/bias must satisfy common-mode and output swing across tolerance; old 3V3/VBOT circuit rejected" (at 25 48 0) (effects (font (size 1.6 1.6)) (justify left)))
-  (text "TIA output -> low-threshold comparator + high-threshold comparator -> active-low FPGA inputs" (at 25 61 0) (effects (font (size 1.6 1.6)) (justify left)))
-  (text "Eight DAC thresholds; RC filtering at each comparator; optional buffered analog monitor/test points" (at 25 74 0) (effects (font (size 1.6 1.6)) (justify left)))
-  (text "Summing-node no-pour keepout and extracted-parasitic stability simulation are release gates" (at 25 87 0) (effects (font (size 1.6 1.6)) (justify left)))
-  (sheet_instances (path "/" (page "3"))) (embedded_fonts no)
+(kicad_sch
+	(version 20260306)
+	(generator "eeschema")
+	(generator_version "10.0")
+	(paper "A3")
+	(title_block
+		(title "Muon3 four-channel analog front end")
+		(date "2026-07-11")
+		(rev "P1")
+		(comment 1 "BASIC SCHEMATIC - WIP")
+	)
 )
