File: pcb/connectors_sensors.kicad_sch (KiCad schematic)
At the start: 0 parts

Commit message: Update paper with latest architecture, add openEMS EM simulations (RF, SI, PDN), update schematics with real symbols/wires, add 3D models and openEMS figures
Other:
- note removed: "BME280 C92489 for atmospheric pressure/humidity/temperature and condensation calculations"
- note removed: "Four polarized locking MPPC/panel interfaces: SiPM bias, signal/return, NTC and Peltier pair"
- note removed: "No exposed connector shell carries HV; optional coax is signal-only with grounded shield"
- note removed: "SWD, FPGA configuration, UART/service USB, spare I2C/SPI and current-limited test points"
Changed lines of the file:
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@@
-(kicad_sch (version 20250114) (generator "eeschema") (generator_version "9.0")
- (paper "A3")
-  (title_block (title "Muon3 panel connectors, sensors and debug") (date "2026-07-11") (rev "P0") (comment 1 "ARCHITECTURE - electrical capture pending"))
-  (text "Four polarized locking MPPC/panel interfaces: SiPM bias, signal/return, NTC and Peltier pair" (at 25 35 0) (effects (font (size 2 2)) (justify left)))
-  (text "No exposed connector shell carries HV; optional coax is signal-only with grounded shield" (at 25 48 0) (effects (font (size 1.6 1.6)) (justify left)))
-  (text "BME280 C92489 for atmospheric pressure/humidity/temperature and condensation calculations" (at 25 61 0) (effects (font (size 1.6 1.6)) (justify left)))
-  (text "SWD, FPGA configuration, UART/service USB, spare I2C/SPI and current-limited test points" (at 25 74 0) (effects (font (size 1.6 1.6)) (justify left)))
-  (sheet_instances (path "/" (page "6"))) (embedded_fonts no)
+(kicad_sch
+	(version 20260306)
+	(generator "eeschema")
+	(generator_version "10.0")
+	(paper "A3")
+	(title_block
+		(title "Muon3 panel connectors, sensors and debug")
+		(date "2026-07-11")
+		(rev "P1")
+		(comment 1 "BASIC SCHEMATIC - WIP")
+	)
 )
