File: pcb/digital_radio.kicad_sch (KiCad schematic)
At the start: 0 parts

Commit message: Update paper with latest architecture, add openEMS EM simulations (RF, SI, PDN), update schematics with real symbols/wires, add 3D models and openEMS figures
Other:
- note removed: "Direct nRF9151-LACA-R7 C22397843: LTE-M/NB-IoT, GNSS, application MCU and housekeeping"
- note removed: "LTE and GNSS RF paths/keepouts follow Nordic reference layout; two grounded-shell antenna connectors"
- note removed: "Nano-SIM plus DNP MFF2 eSIM option; Onomondo/Telekom profile selected per deployment"
- note removed: "SPI flash, 25 MHz TCXO, GNSS PPS to FPGA and MCU, SWD/FPGA programming and test points"
- note removed: "iCE40UP5K-SG48I C2678152: 1V2 VCC/VCCPLL, 3V3 VCCIO, dual thresholds and exact-subset coincidence"
Changed lines of the file:
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@@
-(kicad_sch (version 20250114) (generator "eeschema") (generator_version "9.0")
- (paper "A3")
-  (title_block (title "Muon3 digital, cellular and timing") (date "2026-07-11") (rev "P0") (comment 1 "ARCHITECTURE - electrical capture pending"))
-  (text "Direct nRF9151-LACA-R7 C22397843: LTE-M/NB-IoT, GNSS, application MCU and housekeeping" (at 25 35 0) (effects (font (size 2 2)) (justify left)))
-  (text "Nano-SIM plus DNP MFF2 eSIM option; Onomondo/Telekom profile selected per deployment" (at 25 48 0) (effects (font (size 1.6 1.6)) (justify left)))
-  (text "iCE40UP5K-SG48I C2678152: 1V2 VCC/VCCPLL, 3V3 VCCIO, dual thresholds and exact-subset coincidence" (at 25 61 0) (effects (font (size 1.6 1.6)) (justify left)))
-  (text "SPI flash, 25 MHz TCXO, GNSS PPS to FPGA and MCU, SWD/FPGA programming and test points" (at 25 74 0) (effects (font (size 1.6 1.6)) (justify left)))
-  (text "LTE and GNSS RF paths/keepouts follow Nordic reference layout; two grounded-shell antenna connectors" (at 25 87 0) (effects (font (size 1.6 1.6)) (justify left)))
-  (sheet_instances (path "/" (page "4"))) (embedded_fonts no)
+(kicad_sch
+	(version 20260306)
+	(generator "eeschema")
+	(generator_version "10.0")
+	(paper "A3")
+	(title_block
+		(title "Muon3 digital, cellular and timing")
+		(date "2026-07-11")
+		(rev "P1")
+		(comment 1 "BASIC SCHEMATIC - WIP")
+	)
 )
